File: pcb/untitled.kicad_sch (KiCad schematic)
At the start: 51 parts, among them IC10 AD844_OPAMP_MEL, IC3 FOD814_OPTO_NOSHD, IC5 FOD814_OPTO_MEL, IC6 AD844_OPAMP_AL, IC7 FOD814_OPTO_AL, IC8 AD844_OPAMP_NOSHD, U2 REF192_NOSHD, U3 REF192_AL, U4 REF192_MEL

Commit message: Added more to the BOM
Parts:
- C19, C20, C28, C32, C34, C38: Manufacturer_Name (none) -> KEMET; Manufacturer_Part_Number (none) -> C0805C103K4RACAUTO
- C21, C31, C37: Manufacturer_Part_Number C0805C105Z5VACTU -> C0805C105K4RACAUTO
- C22, C23, C24: Manufacturer_Name KEMET -> Murata; Manufacturer_Part_Number T495D106K035ATE300 -> GRT21BR61C106KE01L
- C29, C30, C35, C36, C39, C40: Manufacturer_Part_Number C0805C224M5VACTU -> C0805C224K4RACAUTO
- R15, R19, R23: Manufacturer_Name (none) -> Panasonic; Manufacturer_Part_Number (none) -> ERJ-2RKF8200X
- R16, R20, R24: Manufacturer_Name (none) -> Panasonic; Manufacturer_Part_Number (none) -> ERJ-2RKF47R0X
- R17, R18, R26, R27, R29, R30: Manufacturer_Name (none) -> Panasonic; Manufacturer_Part_Number (none) -> ERJ-H2RF1000X
- R22, R28, R34: Manufacturer_Name (none) -> Panasonic; Manufacturer_Part_Number (none) -> ERJ-2RKF1003X
- R25, R31, R35: Manufacturer_Name (none) -> Panasonic; Manufacturer_Part_Number (none) -> ERJ-2RKF1001X

Commit message: Finished BOM and fixed file paths for 3D models
Parts:
- J_AD1, J_AD2, J_AD3: now not fitted
- U2, U3, U4: Manufacturer_Name (none) -> Analog Devices; Manufacturer_Part_Number (none) -> REF192GSZ
Changed lines of the file:
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@@
 			)
 		)
+		(property "Manufacturer_Name" "Analog Devices"
+			(at 151.13 125.73 0)
+			(effects
+				(font
+					(size 1.27 1.27)
+				)
+				(hide yes)
+			)
+		)
+		(property "Manufacturer_Part_Number" "REF192GSZ"
+			(at 151.13 125.73 0)
+			(effects
+				(font
+					(size 1.27 1.27)
+				)
+				(hide yes)
+			)
+		)
 		(pin "1"
 		)
@@
 			)
 		)
+		(property "Manufacturer_Name" "Analog Devices"
+			(at 151.13 191.77 0)
+			(effects
+				(font
+					(size 1.27 1.27)
+				)
+				(hide yes)
+			)
+		)
+		(property "Manufacturer_Part_Number" "REF192GSZ"
+			(at 151.13 191.77 0)
+			(effects
+				(font
+					(size 1.27 1.27)
+				)
+				(hide yes)
+			)
+		)
 		(pin "1"
 		)
@@
 		(in_bom yes)
 		(on_board yes)
-		(dnp no)
+		(dnp yes)
 		(fields_autoplaced yes)
 		(property "Reference" "J_AD1"
@@
 		(in_bom yes)
 		(on_board yes)
-		(dnp no)
+		(dnp yes)
 		(fields_autoplaced yes)
 		(property "Reference" "J_AD3"
@@
 		(in_bom yes)
 		(on_board yes)
-		(dnp no)
+		(dnp yes)
 		(fields_autoplaced yes)
 		(property "Reference" "J_AD2"
@@
 			(at 148.59 43.18 0)
 			(effects
+				(font
+					(size 1.27 1.27)
+				)
+				(hide yes)
+			)
+		)
+		(property "Manufacturer_Name" "Analog Devices"
+			(at 148.59 43.18 0)
+			(effects
+				(font
+					(size 1.27 1.27)
+				)
+				(hide yes)
+			)
+		)
+		(property "Manufacturer_Part_Number" "REF192GSZ"
+			(at 148.59 43.18 0)
+			(effects

Commit message: updated component labels
Parts:
- renumbered IC8 to IC1, U2 to IC2, IC6 to IC4, U3 to IC5, IC7 to IC6, IC10 to IC7, U4 to IC8, IC5 to IC9

Commit message: Finished C25 BOM designation
Parts:
- C19, C20, C28, C32, C34, C38: Manufacturer_Part_Number C0805C103K4RACAUTO -> (none)
- C21, C31, C37: Manufacturer_Part_Number C0805C105K4RACAUTO -> (none)
- C22, C23, C24: Manufacturer_Part_Number GRT21BR61C106KE01L -> (none)
- C29, C30, C35, C36, C39, C40: Manufacturer_Part_Number C0805C224K4RACAUTO -> (none)
- IC1, IC4, IC7: Manufacturer_Part_Number AD844JRZ-16-REEL7 -> (none)
- IC2, IC5, IC8: Manufacturer_Part_Number REF192GSZ -> (none)
- IC3, IC6, IC9: Manufacturer_Part_Number FOD814SD -> (none)
- R15, R19, R23: Manufacturer_Part_Number ERJ-2RKF8200X -> (none)
- R16, R20, R24: Manufacturer_Part_Number ERJ-2RKF47R0X -> (none)
- R17, R18, R26, R27, R29, R30: Manufacturer_Part_Number ERJ-H2RF1000X -> (none)
- R22, R28, R34: Manufacturer_Part_Number ERJ-2RKF1003X -> (none)
- R25, R31, R35: Manufacturer_Part_Number ERJ-2RKF1001X -> (none)

Commit message: Started fixing the BOM
Parts:
- IC1, IC4, IC7: MPN (none) -> AD844JRZ-16-REEL7; Manufacturer (none) -> Analog Devices Inc.
- IC2, IC5, IC8: MPN (none) -> REF192GSZ; Manufacturer (none) -> Analog Devices Inc.
- IC3, IC6, IC9: MPN (none) -> FOD814SD; Manufacturer (none) -> onsemi
- R15, R19, R23: MPN (none) -> CRCW0402820RFKED; Manufacturer (none) -> Vishay Dale
- R16, R20, R24: MPN (none) -> CRCW040247R0FKTD; Manufacturer (none) -> Vishay Dale
- R17, R18, R26, R27, R29, R30: MPN (none) -> CRCW0402100RFKTD; Manufacturer (none) -> Vishay Dale
- R22, R28, R34: MPN (none) -> CRCW0402100KFKTD; Manufacturer (none) -> Vishay Dale
- R25, R31, R35: MPN (none) -> CRCW04021K00FKTD; Manufacturer (none) -> Vishay Dale

Commit message: Did more work on the BOM
Parts:
- C19, C20, C28, C32, C34, C38: MPN (none) -> C0805C104J4RALTU; Manufacturer (none) -> KEMET
- C22, C23, C24: MPN (none) -> C0805C106M4RALTU; Manufacturer (none) -> KEMET
Changed lines of the file:
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@@
 			)
 		)
-		(property "Datasheet" "C0805C104K5RAC7210"
+		(property "Datasheet" "https://yageogroup.com/content/datasheet/asset/file/KEM_C1018_X7R_SnPb_SMD"
 			(at 146.05 203.2 0)
 			(hide yes)
@@
 			)
 		)
-		(property "Description" ""
+		(property "Description" "0.1 µF ±5% 16V Ceramic Capacitor X7R 0805 (2012 Metric)"
 			(at 146.05 203.2 0)
 			(hide yes)
@@
 			)
 		)
-		(property "MPN" ""
+		(property "MPN" "C0805C104J4RALTU"
 			(at 146.05 203.2 90)
 			(hide yes)
@@
 			)
 		)
-		(property "Manufacturer" ""
+		(property "Manufacturer" "KEMET"
 			(at 146.05 203.2 90)
 			(hide yes)
@@
 			)
 		)
-		(property "Datasheet" "C0805C104K5RAC7210"
+		(property "Datasheet" "https://yageogroup.com/content/datasheet/asset/file/KEM_C1018_X7R_SnPb_SMD"
 			(at 143.51 54.61 0)
 			(hide yes)
@@
 			)
 		)
-		(property "Description" ""
+		(property "Description" "0.1 µF ±5% 16V Ceramic Capacitor X7R 0805 (2012 Metric)"
 			(at 143.51 54.61 0)
 			(hide yes)
@@
 			)
 		)
-		(property "MPN" ""
+		(property "MPN" "C0805C104J4RALTU"
 			(at 143.51 54.61 90)
 			(hide yes)
@@
 			)
 		)
-		(property "Manufacturer" ""
+		(property "Manufacturer" "KEMET"
 			(at 143.51 54.61 90)
 			(hide yes)
@@
 			)
 		)
-		(property "Datasheet" "C0805C104K5RAC7210"
+		(property "Datasheet" "https://yageogroup.com/content/datasheet/asset/file/KEM_C1018_X7R_SnPb_SMD"
 			(at 208.28 54.61 0)
 			(hide yes)
@@
 			)
 		)
-		(property "Description" ""
+		(property "Description" "0.1 µF ±5% 16V Ceramic Capacitor X7R 0805 (2012 Metric)"
 			(at 208.28 54.61 0)
 			(hide yes)
@@
 			)
 		)
-		(property "MPN" ""
+		(property "MPN" "C0805C104J4RALTU"
 			(at 208.28 54.61 90)
 			(hide yes)
@@
 			)
 		)
-		(property "Manufacturer" ""
+		(property "Manufacturer" "KEMET"
 			(at 208.28 54.61 90)
 			(hide yes)
@@
 			)
 		)
-		(property "Datasheet" "C0805C104K5RAC7210"
+		(property "Datasheet" "https://yageogroup.com/content/datasheet/asset/file/KEM_C1018_X7R_SnPb_SMD"
 			(at 210.82 203.2 0)
 			(hide yes)
@@
 			)
 		)
-		(property "Description" ""
+		(property "Description" "0.1 µF ±5% 16V Ceramic Capacitor X7R 0805 (2012 Metric)"
 			(at 210.82 203.2 0)
 			(hide yes)
@@
 			)
 		)
-		(property "MPN" ""
+		(property "MPN" "C0805C104J4RALTU"
 			(at 210.82 203.2 90)
 			(hide yes)
@@
 			)
 		)
-		(property "Manufacturer" ""
+		(property "Manufacturer" "KEMET"
 			(at 210.82 203.2 90)
 			(hide yes)
@@
 			)
 		)
-		(property "Datasheet" "C0805C104K5RAC7210"
+		(property "Datasheet" "https://yageogroup.com/content/datasheet/asset/file/KEM_C1018_X7R_SnPb_SMD"
 			(at 210.82 137.16 0)
 			(hide yes)
@@
 			)
 		)
-		(property "Description" ""
+		(property "Description" "0.1 µF ±5% 16V Ceramic Capacitor X7R 0805 (2012 Metric)"
 			(at 210.82 137.16 0)
 			(hide yes)
@@
 			)
 		)
-		(property "MPN" ""
+		(property "MPN" "C0805C104J4RALTU"
 			(at 210.82 137.16 90)
 			(hide yes)
@@
 			)
 		)
-		(property "Manufacturer" ""
+		(property "Manufacturer" "KEMET"
 			(at 210.82 137.16 90)
 			(hide yes)
@@
 			)
 		)
-		(property "Datasheet" "https://content.kemet.com/datasheets/KEM_T2009_T495.pdf"
+		(property "Datasheet" "https://yageogroup.com/content/datasheet/asset/file/KEM_C1002_X7R_SMD"
 			(at -60.3 60.96 0)
 			(hide yes)
@@
 			)
 		)
-		(property "Description" ""
+		(property "Description" "10 µF ±10% 10V Ceramic Capacitor X7R 0805 (2012 Metric)"
 			(at 135.89 52.07 0)
 			(hide yes)
@@
 			)
 		)
-		(property "MPN" ""
+		(property "MPN" "C0805C106M4RALTU"
 			(at 135.89 52.07 90)
 			(hide yes)
@@
 			)
 		)
-		(property "Manufacturer" ""
+		(property "Manufacturer" "KEMET"
 			(at 135.89 52.07 90)
 			(hide yes)
@@
 			)
 		)
-		(property "Datasheet" "https://content.kemet.com/datasheets/KEM_T2009_T495.pdf"
+		(property "Datasheet" "https://yageogroup.com/content/datasheet/asset/file/KEM_C1002_X7R_SMD"
 			(at -57.76 209.55 0)
 			(hide yes)
@@
 			)
 		)
-		(property "Description" ""
+		(property "Description" "10 µF ±10% 10V Ceramic Capacitor X7R 0805 (2012 Metric)"
 			(at 138.43 200.66 0)
 			(hide yes)
@@
 			)
 		)
-		(property "MPN" ""
+		(property "MPN" "C0805C106M4RALTU"
 			(at 138.43 200.66 90)
 			(hide yes)
@@
 			)
 		)
-		(property "Manufacturer" ""
+		(property "Manufacturer" "KEMET"
 			(at 138.43 200.66 90)
 			(hide yes)
@@
 			)
 		)
-		(property "Datasheet" "C0805C104K5RAC7210"
+		(property "Datasheet" "https://yageogroup.com/content/datasheet/asset/file/KEM_C1018_X7R_SnPb_SMD"
 			(at 146.05 137.16 0)
 			(hide yes)
@@
 			)
 		)
-		(property "Description" ""
+		(property "Description" "0.1 µF ±5% 16V Ceramic Capacitor X7R 0805 (2012 Metric)"
 			(at 146.05 137.16 0)
 			(hide yes)
@@
 			)
 		)
-		(property "MPN" ""
+		(property "MPN" "C0805C104J4RALTU"
 			(at 146.05 137.16 90)
 			(hide yes)
@@
 			)
 		)
-		(property "Manufacturer" ""
+		(property "Manufacturer" "KEMET"
 			(at 146.05 137.16 90)
 			(hide yes)
@@
 			)
 		)
-		(property "Datasheet" "https://content.kemet.com/datasheets/KEM_T2009_T495.pdf"
+		(property "Datasheet" "https://yageogroup.com/content/datasheet/asset/file/KEM_C1002_X7R_SMD"
 			(at -57.76 143.51 0)
 			(hide yes)
@@
 			)
 		)
-		(property "Description" ""
+		(property "Description" "10 µF ±10% 10V Ceramic Capacitor X7R 0805 (2012 Metric)"
 			(at 138.43 134.62 0)
 			(hide yes)
@@
 			)
 		)
-		(property "MPN" ""
+		(property "MPN" "C0805C106M4RALTU"
 			(at 138.43 134.62 90)
 			(hide yes)
@@
 			)
 		)
-		(property "Manufacturer" ""
+		(property "Manufacturer" "KEMET"
 			(at 138.43 134.62 90)
 			(hide yes)

Commit message: Added ferrite bead
Parts:
- C21, C31, C37: MPN (none) -> C0805C105J4RALTU; Manufacturer (none) -> KEMET
- C29, C30, C35, C36, C39, C40: MPN (none) -> C0805C224J4RALTU; Manufacturer (none) -> KEMET
Changed lines of the file:
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@@
 			)
 		)
-		(property "Description" ""
+		(property "Description" "0.22 µF ±5% 16V Ceramic Capacitor X7R 0805 (2012 Metric)"
 			(at 109.22 48.26 0)
 			(hide yes)
@@
 			)
 		)
-		(property "MPN" ""
+		(property "MPN" "C0805C224J4RALTU"
 			(at 109.22 48.26 90)
 			(hide yes)
@@
 			)
 		)
-		(property "Manufacturer" ""
+		(property "Manufacturer" "KEMET"
 			(at 109.22 48.26 90)
 			(hide yes)
@@
 			)
 		)
-		(property "Description" ""
+		(property "Description" "1 µF ±5% 16V Ceramic Capacitor X7R 0805 (2012 Metric)"
 			(at 200.66 52.07 0)
 			(hide yes)
@@
 			)
 		)
-		(property "MPN" ""
+		(property "MPN" "C0805C105J4RALTU"
 			(at 200.66 52.07 90)
 			(hide yes)
@@
 			)
 		)
-		(property "Manufacturer" ""
+		(property "Manufacturer" "KEMET"
 			(at 200.66 52.07 90)
 			(hide yes)
@@
 			)
 		)
-		(property "Description" ""
+		(property "Description" "1 µF ±5% 16V Ceramic Capacitor X7R 0805 (2012 Metric)"
 			(at 203.2 134.62 0)
 			(hide yes)
@@
 			)
 		)
-		(property "MPN" ""
+		(property "MPN" "C0805C105J4RALTU"
 			(at 203.2 134.62 90)
 			(hide yes)
@@
 			)
 		)
-		(property "Manufacturer" ""
+		(property "Manufacturer" "KEMET"
 			(at 203.2 134.62 90)
 			(hide yes)
@@
 			)
 		)
-		(property "Description" ""
+		(property "Description" "0.22 µF ±5% 16V Ceramic Capacitor X7R 0805 (2012 Metric)"
 			(at 53.34 64.77 0)
 			(hide yes)
@@
 			)
 		)
-		(property "MPN" ""
+		(property "MPN" "C0805C224J4RALTU"
 			(at 53.34 64.77 90)
 			(hide yes)
@@
 			)
 		)
-		(property "Manufacturer" ""
+		(property "Manufacturer" "KEMET"
 			(at 53.34 64.77 90)
 			(hide yes)
@@
 			)
 		)
-		(property "Description" ""
+		(property "Description" "1 µF ±5% 16V Ceramic Capacitor X7R 0805 (2012 Metric)"
 			(at 203.2 200.66 0)
 			(hide yes)
@@
 			)
 		)
-		(property "MPN" ""
+		(property "MPN" "C0805C105J4RALTU"
 			(at 203.2 200.66 90)
 			(hide yes)
@@
 			)
 		)
-		(property "Manufacturer" ""
+		(property "Manufacturer" "KEMET"
 			(at 203.2 200.66 90)
 			(hide yes)
@@
 			)
 		)
-		(property "Description" ""
+		(property "Description" "0.22 µF ±5% 16V Ceramic Capacitor X7R 0805 (2012 Metric)"
 			(at 57.15 213.36 0)
 			(hide yes)
@@
 			)
 		)
-		(property "MPN" ""
+		(property "MPN" "C0805C224J4RALTU"
 			(at 57.15 213.36 90)
 			(hide yes)
@@
 			)
 		)
-		(property "Manufacturer" ""
+		(property "Manufacturer" "KEMET"
 			(at 57.15 213.36 90)
 			(hide yes)
@@
 			)
 		)
-		(property "Description" ""
+		(property "Description" "0.22 µF ±5% 16V Ceramic Capacitor X7R 0805 (2012 Metric)"
 			(at 58.42 142.24 0)
 			(hide yes)
@@
 			)
 		)
-		(property "MPN" ""
+		(property "MPN" "C0805C224J4RALTU"
 			(at 58.42 142.24 90)
 			(hide yes)
@@
 			)
 		)
-		(property "Manufacturer" ""
+		(property "Manufacturer" "KEMET"
 			(at 58.42 142.24 90)
 			(hide yes)
@@
 			)
 		)
-		(property "Description" ""
+		(property "Description" "0.22 µF ±5% 16V Ceramic Capacitor X7R 0805 (2012 Metric)"
 			(at 114.3 125.73 0)
 			(hide yes)
@@
 			)
 		)
-		(property "MPN" ""
+		(property "MPN" "C0805C224J4RALTU"
 			(at 114.3 125.73 90)
 			(hide yes)
@@
 			)
 		)
-		(property "Manufacturer" ""
+		(property "Manufacturer" "KEMET"
 			(at 114.3 125.73 90)
 			(hide yes)
@@
 			)
 		)
-		(property "Description" ""
+		(property "Description" "0.22 µF ±5% 16V Ceramic Capacitor X7R 0805 (2012 Metric)"
 			(at 113.03 196.85 0)
 			(hide yes)
@@
 			)
 		)
-		(property "MPN" ""
+		(property "MPN" "C0805C224J4RALTU"
 			(at 113.03 196.85 90)
 			(hide yes)
@@
 			)
 		)
-		(property "Manufacturer" ""
+		(property "Manufacturer" "KEMET"
 			(at 113.03 196.85 90)
 			(hide yes)
